File: Hardware/Tools/Cartridge/EEPROM32card.sch (EAGLE design)
At the start: 7 parts

Commit message: Upload PDF schematics
Other:
- note added: "EEPROM/EPROM cartridge with solder jumpers for picking memory pinout"
Changed lines of the file:
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@@
 <sheet>
 <plain>
+<text x="-17.78" y="104.14" size="5.08" layer="97">EEPROM/EPROM cartridge
+with solder jumpers for picking memory pinout</text>
 </plain>
 <instances>
