File: Hardware/Tools/Cartridge/MegaProgrammer.sch (EAGLE design)
At the start: 2 parts

Commit message: Upload PDF schematics
Other:
- note added: "Arduino MEGA shield adapter for GameTank cartridges"
Changed lines of the file:
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@@
 <sheet>
 <plain>
+<text x="-73.66" y="91.44" size="6.4516" layer="97">Arduino MEGA shield adapter for GameTank cartridges</text>
 </plain>
 <instances>
