File: Hardware/KiCad/LogicBoard/CPU_and_address_decode.kicad_sch (KiCad schematic)
At the start: 20 parts, among them IC12 7408N, IC16 7404N, IC32 7432N, IC4 7404N, IC53 7404N, IC7 7408N, U1 W65C02SP, U2 VIA

Commit message: merge of some kind from laptop idk
Parts:
- removed VIAPORT0: PINHD-1X14, cpu-blitter-inputs:1X14, symbol cpu-blitter-inputs-eagle-import:PINHD-1X14
- added J1: Conn_01x26_Socket, symbol Connector:Conn_01x26_Socket
Connections:
- net GND: now also J1.9 (Pin_9)
- net VCC: now also J1.10 (Pin_10)
- net ~{RESET}: now also J1.5 (Pin_5)
- net at U2.14 (PB4): now also J1.23 (Pin_23)
- net at U2.15 (PB5): now also J1.24 (Pin_24)
- net at U2.16 (PB6): now also J1.25 (Pin_25)
- net at U2.17 (PB7): now also J1.26 (Pin_26)
- net at U2.5 (PA3): now also J1.11 (Pin_11)
- net at U2.6 (PA4): now also J1.12 (Pin_12)
- net at U2.7 (PA5): now also J1.13 (Pin_13)
- net at U2.8 (PA6): now also J1.14 (Pin_14)
- net at U2.10 (PB0): now also J1.19 (Pin_19)
- net at U2.11 (PB1): now also J1.20 (Pin_20)
- net at U2.12 (PB2): now also J1.21 (Pin_21)
- net at U2.13 (PB3): now also J1.22 (Pin_22)
- net BusEnable: now reaches R5.1, U1.36 (BE)
- net BusEnable: now also J1.6 (Pin_6)
- net A15: now reaches IC4.1 (I), TOPDECODER0.1 (G), U1.25 (A15)
- net A15: now also J1.8 (Pin_8)
- net MemLock: now reaches U1.5 (MLB)
- net MemLock: now also J1.7 (Pin_7)
- net sync: now reaches U1.7 (SYNC)
- net sync: now also J1.2 (Pin_2)
- net at U2.18 (CB1): now also J1.17 (Pin_17)
- net at U2.19 (CB2): now also J1.18 (Pin_18)
- net at U2.39 (CA2): now also J1.16 (Pin_16)
- net at U2.40 (CA1): now also J1.15 (Pin_15)
- new net CLK28: J1.3 (Pin_3)
- new net R/~{W}: J1.1 (Pin_1)
- new net VNMI: J1.4 (Pin_4)
