File: Hardware/KiCad/LogicBoard/cpu-blitter-inputs.kicad_sch (KiCad schematic)
At the start: 0 parts

Commit message: merge of some kind from laptop idk
Other:
- added sheet Power Units (power_units.kicad_sch)
