File: Hardware/KiCad/Controller/controller_v3/gpad1.kicad_pcb (KiCad board)
At the start: 2 copper layers, 130 x 50 mm, 20 parts, among them IC1 74157N, SW1 SW_MEC_5E, SW2 SW_MEC_5E, SW3 SW_MEC_5E, SW4 SW_MEC_5E, SW5 SW_MEC_5E, SW6 SW_MEC_5E, SW7 SW_MEC_5E, SW8 SW_MEC_5E

Commit message: fix for smt controller
Connections:
- R4 pad 1: Net-(SW4-K) -> Net-(IC1A-2B)
- SW1 pad 1: GND -> unconnected-(SW1-Pad1)
- SW1 pad 2: unconnected-(SW1-Pad2) -> GND
- SW4 pad 1: GND -> unconnected-(SW4-Pad1)
- SW4 pad 2: unconnected-(SW4-Pad2) -> GND
- SW4 pad 3: Net-(SW4-K) -> unconnected-(SW4-K-Pad3)
Routing:
- net Net-(IC1A-2B): track 39.3 -> 46.9 mm, vias 0 -> 2
- net Net-(SW4-K): track 5.10 -> 0.00 mm
- net Net-(IC1A-1B): track 65.7 -> 67.7 mm
- net GND: track 26.9 -> 27.5 mm
Other:
- outline, holes or cut-outs redrawn
- board text added: "GameTank Gamepad v3.1 Clyde Shaffer August 2024"
- board text removed: "GameTank Gamepad v3 Clyde Shaffer August 2024"

Commit message: merge of some kind from laptop idk
Other:
- board text added: "WayWayWay"
Changed lines of the file:
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@@
     (effects (font (size 1.63576 1.63576) (thickness 0.14224)) (justify left bottom))
+  )
+  (gr_text "WayWayWay" (at 207.9 128) (layer "F.SilkS")
+    (effects (font (size 1 1) (thickness 0.1)) (justify left bottom))
   )
   (gr_text "9 8 7 6 5 4 3 2 1" (at 175 112.5) (layer "F.SilkS")
