File: Hardware/KiCad/Controller/controller_v3/gpad1.kicad_sch (KiCad schematic)
At the start: 20 parts, among them IC1 74157N, SW1 SW_MEC_5E, SW2 SW_MEC_5E, SW3 SW_MEC_5E, SW4 SW_MEC_5E, SW5 SW_MEC_5E, SW6 SW_MEC_5E, SW7 SW_MEC_5E, SW8 SW_MEC_5E

Commit message: fix for smt controller
Connections:
- net GND: now also SW1.2, SW4.2; no longer SW1.1, SW4.1
- net at SW4.3 (K): no longer R4.1
- net at IC1.6 (2B), SW4.4 (A): now also R4.1
Changed lines of the file:
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@@
   (junction (at 154.94 96.52) (diameter 0) (color 0 0 0 0)
   )
-  (junction (at 30.48 99.06) (diameter 0) (color 0 0 0 0)
-  )
   (junction (at 154.94 116.84) (diameter 0) (color 0 0 0 0)
   )
@@
   (junction (at 91.44 93.98) (diameter 0) (color 0 0 0 0)
   )
+  (junction (at 96.52 99.06) (diameter 0) (color 0 0 0 0)
+  )
   (junction (at 96.52 63.5) (diameter 0) (color 0 0 0 0)
   )
@@
   (junction (at 106.68 116.84) (diameter 0) (color 0 0 0 0)
   )
+  (junction (at 30.48 101.6) (diameter 0) (color 0 0 0 0)
+  )
   (junction (at 91.44 63.5) (diameter 0) (color 0 0 0 0)
   )
@@
     (stroke (width 0.1524) (type solid))
   )
-  (wire (pts (xy 30.48 76.2) (xy 30.48 83.82))
-    (stroke (width 0) (type default))
-  )
-  (wire (pts (xy 96.52 73.66) (xy 96.52 97.79))
+  (wire (pts (xy 30.48 101.6) (xy 50.8 101.6))
+    (stroke (width 0) (type default))
+  )
+  (wire (pts (xy 60.96 99.06) (xy 96.52 99.06))
     (stroke (width 0) (type default))
   )
@@
     (stroke (width 0.1524) (type solid))
   )
-  (wire (pts (xy 30.48 76.2) (xy 50.8 76.2))
-    (stroke (width 0) (type default))
-  )
   (wire (pts (xy 116.84 73.66) (xy 116.84 132.08))
     (stroke (width 0) (type default))
   )
-  (wire (pts (xy 93.98 99.06) (xy 96.52 101.6))
-    (stroke (width 0) (type default))
-  )
   (wire (pts (xy 30.48 106.68) (xy 30.48 114.3))
     (stroke (width 0) (type default))
   )
+  (wire (pts (xy 96.52 73.66) (xy 96.52 99.06))
+    (stroke (width 0) (type default))
+  )
   (wire (pts (xy 154.94 96.52) (xy 154.94 91.44))
     (stroke (width 0.1524) (type solid))
@@
     (stroke (width 0.1524) (type solid))
   )
+  (wire (pts (xy 30.48 78.74) (xy 30.48 83.82))
+    (stroke (width 0) (type default))
+  )
+  (wire (pts (xy 60.96 76.2) (xy 78.74 76.2))
+    (stroke (width 0) (type default))
+  )
   (wire (pts (xy 81.28 78.74) (xy 220.98 78.74))
     (stroke (width 0.1524) (type solid))
@@
     (stroke (width 0.1524) (type solid))
   )
-  (wire (pts (xy 74.93 76.2) (xy 77.47 78.74))
-    (stroke (width 0) (type default))
-  )
   (wire (pts (xy 101.6 109.22) (xy 134.62 109.22))
     (stroke (width 0.1524) (type solid))
@@
     (stroke (width 0.1524) (type solid))
   )
+  (wire (pts (xy 30.48 78.74) (xy 50.8 78.74))
+    (stroke (width 0) (type default))
+  )
   (wire (pts (xy 30.48 83.82) (xy 30.48 91.44))
     (stroke (width 0) (type default))
   )
-  (wire (pts (xy 77.47 78.74) (xy 81.28 78.74))
-    (stroke (width 0) (type default))
-  )
   (wire (pts (xy 106.68 73.66) (xy 106.68 116.84))
     (stroke (width 0) (type default))
@@
     (stroke (width 0.1524) (type solid))
   )
-  (wire (pts (xy 62.23 102.87) (xy 92.71 102.87))
-    (stroke (width 0) (type default))
-  )
-  (wire (pts (xy 30.48 91.44) (xy 30.48 99.06))
-    (stroke (width 0) (type default))
-  )
   (wire (pts (xy 30.48 106.68) (xy 50.8 106.68))
     (stroke (width 0) (type default))
@@
     (stroke (width 0.1524) (type solid))
   )
+  (wire (pts (xy 96.52 99.06) (xy 96.52 101.6))
+    (stroke (width 0) (type default))
+  )
   (wire (pts (xy 111.76 73.66) (xy 111.76 124.46))
     (stroke (width 0) (type default))
@@
     (stroke (width 0.1524) (type solid))
   )
-  (wire (pts (xy 60.96 99.06) (xy 93.98 99.06))
-    (stroke (width 0) (type default))
-  )
   (wire (pts (xy 60.96 116.84) (xy 106.68 116.84))
     (stroke (width 0.1524) (type solid))
@@
     (stroke (width 0.1524) (type solid))
   )
-  (wire (pts (xy 62.23 102.87) (xy 60.96 101.6))
-    (stroke (width 0) (type default))
-  )
   (wire (pts (xy 203.2 99.06) (xy 220.98 99.06))
     (stroke (width 0.1524) (type solid))
@@
     (stroke (width 0.1524) (type solid))
   )
+  (wire (pts (xy 78.74 76.2) (xy 81.28 78.74))
+    (stroke (width 0) (type default))
+  )
   (wire (pts (xy 154.94 121.92) (xy 154.94 116.84))
     (stroke (width 0.1524) (type solid))
   )
+  (wire (pts (xy 30.48 101.6) (xy 30.48 106.68))
+    (stroke (width 0) (type default))
+  )
   (wire (pts (xy 30.48 121.92) (xy 30.48 129.54))
     (stroke (width 0) (type default))
@@
     (stroke (width 0.1524) (type solid))
   )
-  (wire (pts (xy 60.96 76.2) (xy 74.93 76.2))
-    (stroke (width 0) (type default))
-  )
   (wire (pts (xy 198.12 86.36) (xy 203.2 81.28))
     (stroke (width 0.1524) (type solid))
@@
     (stroke (width 0.1524) (type solid))
   )
-  (wire (pts (xy 30.48 99.06) (xy 50.8 99.06))
-    (stroke (width 0) (type default))
-  )
   (wire (pts (xy 60.96 93.98) (xy 91.44 93.98))
     (stroke (width 0.1524) (type solid))
@@
     (stroke (width 0.1524) (type solid))
   )
-  (wire (pts (xy 30.48 99.06) (xy 30.48 106.68))
+  (wire (pts (xy 30.48 91.44) (xy 30.48 101.6))
     (stroke (width 0) (type default))
   )
@@
     (stroke (width 0.1524) (type solid))
   )
-  (wire (pts (xy 96.52 97.79) (xy 92.71 102.87))
-    (stroke (width 0) (type default))
-  )
   (wire (pts (xy 220.98 88.9) (xy 233.68 88.9))
