File: Hardware/KiCad/LogicBoard_smt/LogicBoard_smt.kicad_sch (KiCad schematic)
At the start: 0 parts

Commit message: manual and models and misc hardware file updates
Other:
- added sheet Power (power.kicad_sch)
Changed lines of the file:
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@@
+    )
+  )
+  (sheet (at 102.87 80.01) (size 53.34 44.45) (fields_autoplaced)
+    (stroke (width 0.1524) (type solid))
+    (fill (color 0 0 0 0.0000))
+    (property "Sheetname" "Power" (at 102.87 79.2984 0)
+      (effects (font (size 1.27 1.27)) (justify left bottom))
+    )
+    (property "Sheetfile" "power.kicad_sch" (at 102.87 125.0446 0)
+      (effects (font (size 1.27 1.27)) (justify left top))
+    )
+    (instances
+      (project "LogicBoard_smt"
+        (path "/28034957-81b4-48a5-b869-6f4cb8f0c2fa" (page "8"))
+      )
     )
   )
