File: Hardware/KiCad/LogicBoard_smt/cpu-blitter-inputs_5.kicad_sch (KiCad schematic)
At the start: 1 part

Commit message: collect production documents for quoting
Parts:
- TO_AUDIO_PROCESSOR1: footprint Connector_FFC-FPC:TE_4-1734839-0_1x40-1MP_P0.5mm_Horizontal -> SamacSys_Parts:F34G1A7Q1E8C40; MPN 4-1734839-0 -> F34G-1A7Q1-E8C40
