File: Hardware/KiCad/LogicBoard_smt/LogicBoard_smt.kicad_pcb (KiCad board)
At the start: 4 copper layers, 177.8 x 168.9 mm, 157 parts, among them IC1 7408N, IC12 7408N, IC16 7404N, IC18 7432N, IC2 AP63205WU-7, IC20 7430N, IC21 7400N, IC3 74573N, IC31 7400N, IC32 7432N, IC4 7404N, IC5 7400N, IC53 7404N, IC7 7408N, IC9 7474N, J1 Conn_01x26_Socket, J2 JACK-PLUG0, J3 Conn_01x03_Pin, U1 W65C02SP, U2 VIA, U3 GFXL, U4 GFXH, U5 GFYL, U6 GFYH, U7 74LVC2G07

Commit message: collect production documents for quoting
Parts:
- removed J3: Conn_01x03_Pin, Connector_PinHeader_1.27mm:PinHeader_1x03_P1.27mm_Vertical
- added U8: MCP130-xxxxTT, Package_TO_SOT_SMD:SOT-23, F.Cu at (192.5, 144.0)
- TO_AUDIO_PROCESSOR1, TO_FRAMEBUFFER1: footprint Connector_FFC-FPC:TE_4-1734839-0_1x40-1MP_P0.5mm_Horizontal -> SamacSys_Parts:F34G1A7Q1E8C40
- moved TO_FRAMEBUFFER1 1.01 mm to (44.0, 66.7)
- moved TO_AUDIO_PROCESSOR1 1.00 mm to (205.0, 66.7)
Routing:
- net GND: track 258.6 -> 277.3 mm
- net unconnected-(U1-NC-Pad35)_1: track 15.4 -> 0.00 mm, vias 2 -> 0
- net VCC: track 309.3 -> 319.5 mm
- net /CPU and address decode/~{RESET}: track 196.5 -> 204.1 mm
Other:
- board text added: "GameTank CPU Board (SMT ver. 3)"
- board text added: "September 2025 - Clyde H. Shaffer III"
- board text removed: "DS1813"
- board text removed: "December 2023 - Clyde H. Shaffer III"
- board text removed: "GameTank CPU Board (SMT ver. 2)"

Commit message: updates
Parts:
- JP1, LED1, RESET_SW_HDR0: footprint Connector_PinHeader_2.54mm:PinHeader_1x02_P2.54mm_Vertical_SMD_Pin1Right -> Connector_PinHeader_2.54mm:PinHeader_1x02_P2.54mm_Vertical
Routing:
- net GND: track 277.3 -> 281.8 mm
- net /CPU and address decode/~{RESET}: track 204.1 -> 199.7 mm
- net Net-(D1-A): track 10.3 -> 12.8 mm
- net Net-(LED1-A): track 5.19 -> 7.37 mm
- net Net-(J2-Pad1): track 38.7 -> 39.6 mm
Other:
- outline, holes or cut-outs redrawn
- board text added: "+"
- board text added: "December 2025 - Clyde H. Shaffer III"
- board text added: "GameTank CPU Board (SMT ver. 4)"
- board text removed: "GameTank CPU Board (SMT ver. 3)"
- board text removed: "September 2025 - Clyde H. Shaffer III"
