File: Hardware/KiCad/LogicBoard_smt/power.kicad_sch (KiCad schematic)
At the start: 10 parts, among them IC2 AP63205WU-7, J2 JACK-PLUG0

Commit message: updates
Parts:
- JP1: footprint Connector_PinHeader_2.54mm:PinHeader_1x02_P2.54mm_Vertical_SMD_Pin1Right -> Connector_PinHeader_2.54mm:PinHeader_1x02_P2.54mm_Vertical; MPN TSM-102-01-L-SV-TR -> G800WC306018EU
Changed lines of the file:
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@@
 			)
 		)
-		(property "Footprint" "Connector_PinHeader_2.54mm:PinHeader_1x02_P2.54mm_Vertical_SMD_Pin1Right"
+		(property "Footprint" "Connector_PinHeader_2.54mm:PinHeader_1x02_P2.54mm_Vertical"
 			(at 106.68 83.82 0)
 			(effects
@@
 			)
 		)
-		(property "MPN" "TSM-102-01-L-SV-TR"
+		(property "MPN" "G800WC306018EU "
 			(at 106.68 83.82 0)
 			(effects
