File: Hardware/KiCad/LogicBoard_smt/CPU_and_address_decode.kicad_sch (KiCad schematic)
At the start: 38 parts, among them IC12 7408N, IC32 7432N, IC4 7404N, IC53 7404N, IC7 7408N, J1 Conn_01x26_Socket, U1 W65C02SP, U2 VIA, U8 MCP130-xxxxTT

Commit message: via irq fix
Parts:
- removed R3: 3.3k, Resistor_SMD:R_0805_2012Metric, symbol cpu-blitter-inputs-eagle-import:R-US_0207/10
- added U7: 74LVC2G07, Package_TO_SOT_SMD:SOT-363_SC-70-6, symbol 74xGxx:74LVC2G07
Connections:
- net ~{IRQ}: now also U7.6; no longer U2.21 (IRQB)
- new net: U2.21 (IRQB), U7.1
