File: Hardware/KiCad/LogicBoard_smt/Gamepad_ports.kicad_sch (KiCad schematic)
At the start: 11 parts

Commit message: via irq fix
Parts:
- PAD1REG0, PAD2REG0: MPN SN74HC573APWR -> SN74AHC573PWR
Changed lines of the file:
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@@
 			)
 		)
-		(property "MPN" "SN74HC573APWR"
+		(property "MPN" "SN74AHC573PWR"
 			(at 137.16 147.32 0)
 			(hide yes)
@@
 			)
 		)
-		(property "MPN" "SN74HC573APWR"
+		(property "MPN" "SN74AHC573PWR"
 			(at 59.69 181.61 0)
 			(hide yes)
@@
 			)
 		)
-		(property "MPN" "SN74HC573APWR"
+		(property "MPN" "SN74AHC573PWR"
 			(at 137.16 81.28 0)
 			(hide yes)
@@
 			)
 		)
-		(property "MPN" "SN74HC573APWR"
+		(property "MPN" "SN74AHC573PWR"
 			(at 43.18 181.61 0)
 			(hide yes)
