File: Hardware/KiCad/LogicBoard_smt/cpu-blitter-inputs_6.kicad_sch (KiCad schematic)
At the start: 14 parts, among them IC16 MC74HC1GU04DFT1G

Commit message: via irq fix
Parts:
- U$6: MPN CD74AC163M96 -> CD74AC161M96
Changed lines of the file:
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@@
 			)
 		)
-		(property "MPN" "CD74AC163M96"
+		(property "MPN" "CD74AC161M96"
 			(at 160.02 96.52 0)
 			(hide yes)
@@
 			)
 		)
-		(property "MPN" "CD74AC163M96"
+		(property "MPN" "CD74AC161M96"
 			(at 196.85 153.67 0)
 			(hide yes)
