File: Hardware/KiCad/AVBoard_smt/signals_4.kicad_sch (KiCad schematic)
At the start: 33 parts, among them IC2_AUD0 7432N, IC4_AUD0 7400N, IC6_AUD0 7474N, IC7_AUD0 LM358N, J4 62684-502100ALF, U1 W65C02SP

Commit message: WIP v2 THT AVboard
Parts:
- AUDJACK0: value RCJ-012 -> RCJ-013; MPN RCJ-012 -> RCJ-013
Changed lines of the file:
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@@
 			)
 		)
-		(property "Value" "RCJ-012"
+		(property "Value" "RCJ-013"
 			(at 530.863 36.8223 0)
 			(show_name no)
@@
 			)
 		)
-		(property "MPN" "RCJ-012"
+		(property "MPN" "RCJ-013"
 			(at 528.32 43.18 0)
 			(hide yes)
