File: Hardware/KiCad/LogicBoard_tht2/CPU_and_address_decode.kicad_sch (KiCad schematic)
At the start: 21 parts, among them IC12 7408N, IC16 7404N, IC32 7432N, IC4 7404N, IC53 7404N, IC7 7408N, J1 Conn_01x26_Socket, U1 W65C02SP, U2 VIA, U3 MCP100-475D

Commit message: new through hole motherboard version
Parts:
- IC12, IC7: DigiKey (none) -> 296-1570-5-ND; MPN (none) -> SN74HC08N
- IC16, IC4, IC53: DigiKey (none) -> 296-1566-5-ND; MPN (none) -> SN74HC04N
- IC32: DigiKey (none) -> 296-1589-5-ND; MPN (none) -> SN74HC32N
- J1: value Conn_01x26_Socket -> DE26; DigiKey (none) -> HDL26-SL-B; MPN (none) -> HDL26-SL-B
- R1, R2, R3, R4, R5: DigiKey (none) -> CF14JT3K30CT-ND; MPN (none) -> CF14JT3K30
- RESET_SW_HDR0: MPN (none) -> DNI*
- TOPDECODER0: DigiKey (none) -> 296-8230-5-ND; MPN (none) -> SN74HC139N
- U$3: DigiKey (none) -> 5530843-3; MPN (none) -> 5530843-3
- U$5: DigiKey (none) -> AS7C256C-15PCN; MPN (none) -> AS7C256C-15PCN
- U1: MPN (none) -> W65C02S6TPG-14; Mouser (none) -> 955-W65C02S6TPG-14; Sourcing (none) -> Direct
- U2: MPN (none) -> W65C22S6TPG-14; Mouser (none) -> 955-W65C22S6TPG-14; Sourcing (none) -> Direct
- U3: DigiKey (none) -> MCP130-475DI/TO-ND; MPN (none) -> MCP130-475DI/TO
- WR_REG_DECODE0: DigiKey (none) -> 2156-CD74HC238EE4-ND; MPN (none) -> CD74HC238EE4; Sourcing (none) -> Rochester
