File: Hardware/KiCad/LogicBoard_tht2/DMA_Controller.kicad_sch (KiCad schematic)
At the start: 47 parts, among them IC1 7408N, IC18 7432N, IC20 7430N, IC21 7400N, IC3 74573N, IC31 7400N, IC32 7432N, IC5 7400N, IC53 7404N, IC54 7407N, IC9 7474N, J2 TX25-40P-6ST-H1E

Commit message: new through hole motherboard version
Parts:
- BANKMUX0, GMUX0, GMUX1, GMUX2, GMUX3, VMUX0, VMUX1, VMUX2, VMUX3: DigiKey (none) -> 296-8285-5-ND; MPN (none) -> SN74HC257N
- BLIT_BUS_SWITCH0: DigiKey (none) -> SN74HC640N; MPN (none) -> SN74HC640N
- BLIT_REG_SELECTOR0: DigiKey (none) -> 2156-CD74HC238EE4-ND; MPN (none) -> CD74HC238EE4; Sourcing (none) -> Rochester
- CLK.SEQ0, IC1: DigiKey (none) -> 296-1570-5-ND; MPN (none) -> SN74HC08N
- CTR.H0, CTR.W0: DigiKey (none) -> CD74HC40103E; MPN (none) -> CD74HC40103E
- GXFLIPPER0, GYFLIPPER0: DigiKey (none) -> SN74AHC8541N; MPN (none) -> SN74AHC8541N
- GXH0, GXL0, GYH0, GYL0, VXH0, VXL0, VYH0, VYL0: DigiKey (none) -> 296-8246-5-ND; MPN (none) -> SN74HC163N
- IC18, IC32: DigiKey (none) -> 296-1589-5-ND; MPN (none) -> SN74HC32N
- IC20: DigiKey (none) -> 296-9196-5-ND; MPN (none) -> CD74HC30E
- IC21, IC31, IC5: DigiKey (none) -> 296-1563-5-ND; MPN (none) -> SN74HC00N
- IC3, REG.COLOR0, REG.FLAGS0, REG.GX0, REG.GY0, REG.H0, REG.VX0, REG.VY0, REG.W0: DigiKey (none) -> 296-12815-5-ND; MPN (none) -> CD74HC573E
- IC53: DigiKey (none) -> 296-1566-5-ND; MPN (none) -> SN74HC04N
- IC54: DigiKey (none) -> 296-14878-5-ND; MPN (none) -> SN74LS07N
- IC9, TRIGGER.INIT0: DigiKey (none) -> 296-1602-5-ND; MPN (none) -> SN74HC74N
- J2: DigiKey (none) -> 670-1446-ND; MPN (none) -> TX25-40P-8ST-H1E
- SEQGEN_XOR0: DigiKey (none) -> 296-8375-5-ND; MPN (none) -> SN74HC86N
- U$4: DigiKey (none) -> AS6C4008-55PCN; MPN (none) -> AS6C4008-55PCN
