File: Hardware/KiCad/LogicBoard_tht2/Gamepad_ports.kicad_sch (KiCad schematic)
At the start: 9 parts

Commit message: new through hole motherboard version
Parts:
- EXTRA_BUTTON_1, EXTRA_BUTTON_2: MPN (none) -> DNI*
- GAMEPAD_SELECTOR0: DigiKey (none) -> 296-1602-5-ND; MPN (none) -> SN74HC74N
- PAD1REG0, PAD2REG0: DigiKey (none) -> 296-12815-5-ND; MPN (none) -> CD74HC573E
- PORT1, PORT2: DigiKey (none) -> LD09P13A4GX00LF; MPN (none) -> LD09P13A4GX00LF
- R6, R7: DigiKey (none) -> CF14JT3K30CT-ND; MPN (none) -> CF14JT3K30
