File: Hardware/KiCad/LogicBoard_tht2/cpu-blitter-inputs_3.kicad_sch (KiCad schematic)
At the start: 69 parts

Commit message: new through hole motherboard version
Parts:
- +5V0, GROUND0, LED1: MPN (none) -> DNI
- C1, C10, C11, C12, C13, C14, C15, C16, C17, C18, C19, C2, C20, C21, C22, C23, C24, C25, C26, C27, C28, C29, C3, C30, C31, C32, C33, C34, C35, C36, C38, C39, C4, C40, C41, C42, C43, C44, C45, C46, C5, C57, C6, C7, C8, C9: value C-US025-024X044 -> 0.1uF
- R16: DigiKey (none) -> CF14JT150RCT-ND; MPN (none) -> CF14JT150R
