File: Hardware/KiCad/LogicBoard_tht2/cpu-blitter-inputs_5.kicad_sch (KiCad schematic)
At the start: 1 part

Commit message: new through hole motherboard version
Parts:
- AUDIOSLOT0: DigiKey (none) -> 670-1385-ND; MPN (none) -> TX24-40R-6ST-N1E
Changed lines of the file:
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@@
+			)
+		)
+		(property "MPN" "TX24-40R-6ST-N1E"
+			(at 195.58 121.92 0)
+			(hide yes)
+			(show_name no)
+			(do_not_autoplace no)
+			(effects
+				(font
+					(size 1.27 1.27)
+				)
+			)
+		)
+		(property "DigiKey" "670-1385-ND"
+			(at 195.58 121.92 0)
+			(hide yes)
+			(show_name no)
+			(do_not_autoplace no)
+			(effects
+				(font
+					(size 1.27 1.27)
+				)
+			)
+		)
+		(property "Mouser" ""
+			(at 195.58 121.92 0)
+			(hide yes)
+			(show_name no)
+			(do_not_autoplace no)
+			(effects
+				(font
+					(size 1.27 1.27)
+				)
+			)
+		)
+		(property "Sourcing" ""
+			(at 195.58 121.92 0)
+			(hide yes)
+			(show_name no)
+			(do_not_autoplace no)
+			(effects
+				(font
+					(size 1.27 1.27)
+				)
 			)
 		)
