File: Hardware/KiCad/LogicBoard_tht2/power_units.kicad_sch (KiCad schematic)
At the start: 1 part

Commit message: new through hole motherboard version
Parts:
- BANKMUX0: DigiKey (none) -> 296-8285-5-ND; MPN (none) -> SN74HC257N
Changed lines of the file:
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@@
+			)
+		)
+		(property "MPN" "SN74HC257N"
+			(at 19.05 24.13 0)
+			(hide yes)
+			(show_name no)
+			(do_not_autoplace no)
+			(effects
+				(font
+					(size 1.27 1.27)
+				)
+			)
+		)
+		(property "DigiKey" "296-8285-5-ND"
+			(at 19.05 24.13 0)
+			(hide yes)
+			(show_name no)
+			(do_not_autoplace no)
+			(effects
+				(font
+					(size 1.27 1.27)
+				)
+			)
+		)
+		(property "Mouser" ""
+			(at 19.05 24.13 0)
+			(hide yes)
+			(show_name no)
+			(do_not_autoplace no)
+			(effects
+				(font
+					(size 1.27 1.27)
+				)
+			)
+		)
+		(property "Sourcing" ""
+			(at 19.05 24.13 0)
+			(hide yes)
+			(show_name no)
+			(do_not_autoplace no)
+			(effects
+				(font
+					(size 1.27 1.27)
+				)
 			)
 		)
