File: Hardware/KiCad/ps_slash_2/ps2mkb/ps2mkb.kicad_sch (KiCad schematic)
At the start: 14 parts, among them J1 Mini-DIN-6, J2 Mini-DIN-6, J3 Conn_01x26_Shielded, U1 74HC595, U10 74HC04, U11 74LS161, U2 74HC595, U3 74HC165, U4 74HC165, U5 74HC03, U6 74HC04, U7 74HC280, U8 74LS32, U9 74HC74

Commit message: update label on part in ps/2 adapter
Parts:
- U11: value 74LS161 -> 74HC161
- U8: value 74LS32 -> 74HC32
Changed lines of the file:
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@@
 			)
 		)
-		(property "Value" "74LS161"
+		(property "Value" "74HC161"
 			(at 200.2633 233.68 0)
 			(show_name no)
@@
 			)
 		)
-		(property "Value" "74LS32"
+		(property "Value" "74HC32"
 			(at 381 43.18 0)
 			(show_name no)
@@
 			)
 		)
-		(property "Value" "74LS32"
+		(property "Value" "74HC32"
 			(at 247.65 76.2 0)
 			(show_name no)
@@
 			)
 		)
-		(property "Value" "74LS32"
+		(property "Value" "74HC32"
 			(at 328.93 92.71 0)
 			(show_name no)
@@
 			)
 		)
-		(property "Value" "74LS32"
+		(property "Value" "74HC32"
 			(at 293.37 168.9099 90)
 			(show_name no)

Commit message: mouse keyboard adapter v1
Parts:
- removed J2: Mini-DIN-6, symbol Connector:Mini-DIN-6
- removed J3: Conn_01x26_Shielded, symbol Connector_Generic_Shielded:Conn_01x26_Shielded
- removed U10: 74HC04, symbol 74xx:74HC04
- removed U11: 74HC161, symbol 74xx:74LS161
- removed U8: 74HC32, symbol 74xx:74LS32
- added CONN_HOST1: Conn_01x26_Shielded, Library:DB26MALE, symbol Connector_Generic_Shielded:Conn_01x26_Shielded
- added CONN_NEXT1: Conn_01x26_Shielded, Library:HDL26-SL-B, symbol Connector_Generic_Shielded:Conn_01x26_Shielded
- added J1: Conn_01x16_Socket, Connector_PinHeader_2.54mm:PinHeader_1x16_P2.54mm_Vertical, symbol Connector:Conn_01x16_Socket
- added PacketClockHigh1, PacketClockLow1: 74HC164, Package_DIP:DIP-14_W7.62mm, symbol 74xx:74HC164
- added R1, R2: R_US, Resistor_THT:R_Axial_DIN0204_L3.6mm_D1.6mm_P7.62mm_Horizontal, symbol Device:R_US
- added RN1: R_Network08 47k, Resistor_THT:R_Array_SIP9, symbol Device:R_Network08
- added SW1: SW_DIP_x08, Button_Switch_THT:SW_DIP_SPSTx08_Slide_9.78x22.5mm_W7.62mm_P2.54mm, symbol Switch:SW_DIP_x08
- added U1: 74HC126, Package_DIP:DIP-14_W7.62mm, symbol 74xx:74LS126
- added U11: 74HC32, Package_DIP:DIP-14_W7.62mm, symbol 74xx:74LS32
- added U2, U4: 74HC573, Package_DIP:DIP-20_W7.62mm, symbol 74xx:74LS573
- added U3: 74HC688, Package_DIP:DIP-20_W7.62mm, symbol 74xx:74HC688
- CONNPS2: renamed from J1; footprint (none) -> Library:MiniDin6; MPN (none) -> KMDGX-6S-BS
- InRegHigh1: renamed from U2; footprint (none) -> Package_DIP:DIP-16_W7.62mm
- InRegLow1: renamed from U1; footprint (none) -> Package_DIP:DIP-16_W7.62mm
- OutRegHigh1: renamed from U3; footprint (none) -> Package_DIP:DIP-16_W7.62mm
- OutRegLow1: renamed from U4; footprint (none) -> Package_DIP:DIP-16_W7.62mm
- ParityGen1: renamed from U7; footprint (none) -> Package_DIP:DIP-14_W7.62mm
- U5, U6, U9: footprint (none) -> Package_DIP:DIP-14_W7.62mm
Connections:
- net ~{OutRegLoad} is gone; now on net PA4: OutRegHigh1.1 (~{PL}), OutRegLow1.1 (~{PL})
- net GND: now also CONN_HOST1.9 (Pin_9), CONN_HOST1.SH (Shield), CONN_NEXT1.9 (Pin_9), CONN_NEXT1.SH (Shield), J1.2 (Pin_2), PacketClockHigh1.7 (GND), PacketClockLow1.7 (GND), SW1.1, SW1.2, SW1.3, SW1.4, SW1.5, SW1.6, SW1.7, SW1.8, U2.1 (OE), U2.10 (GND), U3.10 (GND), U4.10 (GND), U4.2 (D0), U4.4 (D2), U4.5 (D3); no longer U9.3 (C)
- net PA3: now also InRegHigh1.12 (RCLK), InRegHigh1.13 (~{OE}), InRegLow1.12 (RCLK), InRegLow1.13 (~{OE}), U11.3; no longer U9.4 (~{S})
- net PA4: now also U9.10 (~{S}), U11.6; no longer U5.10
- net PA5: now also PacketClockHigh1.9 (~{MR}), PacketClockLow1.9 (~{MR}), U11.8; no longer U9.10 (~{S})
- net PA6: now also InRegHigh1.11 (SRCLK), InRegLow1.11 (SRCLK), U5.2, U6.11, U6.13, PacketClockHigh1.5 (Q2), U1.2
- net PB0: now also CONN_HOST1.19 (Pin_19), CONN_NEXT1.19 (Pin_19), J1.9 (Pin_9), U2.2 (D0), U4.19 (Q0)
- net PB1: now also CONN_HOST1.20 (Pin_20), CONN_NEXT1.20 (Pin_20), J1.10 (Pin_10), U2.3 (D1), U4.18 (Q1)
- net PB2: now also CONN_HOST1.21 (Pin_21), CONN_NEXT1.21 (Pin_21), J1.11 (Pin_11), U2.4 (D2), U4.17 (Q2)
- net PB3: now also CONN_HOST1.22 (Pin_22), CONN_NEXT1.22 (Pin_22), J1.12 (Pin_12), U2.5 (D3), U4.16 (Q3)
- net PB4: now also CONN_HOST1.23 (Pin_23), CONN_NEXT1.23 (Pin_23), J1.13 (Pin_13), U2.6 (D4), U4.15 (Q4)
- net PB5: now also CONN_HOST1.24 (Pin_24), CONN_NEXT1.24 (Pin_24), J1.14 (Pin_14), U2.7 (D5), U4.14 (Q5)
- net PB6: now also CONN_HOST1.25 (Pin_25), CONN_NEXT1.25 (Pin_25), J1.15 (Pin_15), U2.8 (D6), U4.13 (Q6)
- net PB7: now also CONN_HOST1.26 (Pin_26), CONN_NEXT1.26 (Pin_26), J1.16 (Pin_16), U2.9 (D7), U4.12 (Q7)
- net VCC: now also ParityGen1.14 (VCC), U5.1, CONN_HOST1.10 (Pin_10), CONN_NEXT1.10 (Pin_10), J1.1 (Pin_1), PacketClockHigh1.14 (VCC), PacketClockHigh1.2 (DSB), PacketClockLow1.14 (VCC), PacketClockLow1.2 (DSB), R1.2, R2.2, RN1.1 (common), U2.20 (VCC), U3.20 (VCC), U4.11 (Load), U4.20 (VCC), U4.3 (D1), U4.6 (D4), U4.7 (D5), U4.8 (D6), U4.9 (D7)
- net at U6.8: now also U5.12
- net at U5.11: now also R2.1, U4.1 (OE); no longer U6.9
- net at U6.10: now also OutRegHigh1.2 (CP), OutRegLow1.2 (CP), PacketClockHigh1.8 (CP), PacketClockLow1.8 (CP); no longer U6.13
- net at CONNPS2.1, U5.6: now also InRegHigh1.14 (SER), U6.1; no longer U6.5
- net at U6.6: now also U2.11 (Load)
- net at InRegHigh1.10 (~{SRCLR}): now also InRegLow1.10 (~{SRCLR})
- net at U9.13 (~{R}): now also U6.12
- net CA2: now reaches U5.9
- net CA2: now also U5.13, CONN_HOST1.16 (Pin_16), CONN_NEXT1.16 (Pin_16), J1.7 (Pin_7), U11.13; no longer U5.1
- net at U5.8: now also U6.5, R1.1
- net at InRegLow1.2 (QC): no longer U6.1
- removed net OutClock: OutRegHigh1.2 (CP), OutRegLow1.2 (CP), U6.4
- net ~{ChunkStop}: no longer names the net of U9.1 (~{R})
- net ~{ChunkStop}: no longer U6.2
- new net: U2.15 (Q4), U3.11 (P4)
- new net: RN1.5 (R4), SW1.12, U3.12 (R4)
- new net: U2.14 (Q5), U3.13 (P5)
- new net: RN1.4 (R3), SW1.11, U3.14 (R5)
- new net: U2.13 (Q6), U3.15 (P6)
- new net: RN1.3 (R2), SW1.10, U3.16 (R6)
- new net: U2.12 (Q7), U3.17 (P7)
- new net: RN1.2 (R1), SW1.9, U3.18 (R7)
- new net: U11.12, U3.19 (P=R), U6.9
- new net: U2.19 (Q0), U3.2 (P0)
- new net: RN1.9 (R8), SW1.16, U3.3 (R0)
- new net: U2.18 (Q1), U3.4 (P1)
- new net: RN1.8 (R7), SW1.15, U3.5 (R1)
- new net: U2.17 (Q2), U3.6 (P2)
- new net: RN1.7 (R6), SW1.14, U3.7 (R2)
- new net: U2.16 (Q3), U3.8 (P3)
- new net: RN1.6 (R5), SW1.13, U3.9 (R3)
- new net: U11.1, U11.11, U11.4, U11.9, U6.3
- new net: CONN_HOST1.11 (Pin_11), CONN_NEXT1.11 (Pin_11), J1.3 (Pin_3), U11.2
- new net: CONN_HOST1.12 (Pin_12), CONN_NEXT1.12 (Pin_12), J1.4 (Pin_4), U11.5
- new net: CONN_HOST1.13 (Pin_13), CONN_NEXT1.13 (Pin_13), J1.5 (Pin_5), U11.10
- new net: CONN_HOST1.14 (Pin_14), CONN_NEXT1.14 (Pin_14), J1.6 (Pin_6), U1.3
- new net: U1.1, U6.4
- new net: U5.4, U9.9 (Q)
- new net: OutRegHigh1.7 (~{Q7}), U5.5
- new net: PacketClockLow1.1 (DSA), U6.2
- new net: PacketClockHigh1.1 (DSA), PacketClockLow1.13 (Q7)
- new net CB2: CONN_HOST1.18 (Pin_18), CONN_NEXT1.18 (Pin_18), J1.8 (Pin_8), U3.1 (G), U5.10
Other:
- note added: "Address Comparator"
- note added: "Last Published Address"
- note added: "PA3 - Read PA4 - Write PA5 - InhibitClear PA6 - PacketDone"
- note added: "Stack connector"
- note added: "Type Identifier"
- moved on the sheet: CONNPS2, InRegHigh1, InRegLow1, OutRegHigh1, OutRegLow1, ParityGen1, U5A, U5B, U6A, U6B, U9A, U9B

Commit message: backplane and updated mouse keyboard adapter
Parts:
- removed CONN_HOST1: Conn_01x26_Shielded, Library:DB26MALE, symbol Connector_Generic_Shielded:Conn_01x26_Shielded
- removed CONN_NEXT1: Conn_01x26_Shielded, Library:HDL26-SL-B, symbol Connector_Generic_Shielded:Conn_01x26_Shielded
- removed J1: Conn_01x16_Socket, Connector_PinHeader_2.54mm:PinHeader_1x16_P2.54mm_Vertical, symbol Connector:Conn_01x16_Socket
- removed U1: 74HC126, Package_DIP:DIP-14_W7.62mm, symbol 74xx:74LS126
- added D1: LED, LED_THT:LED_D3.0mm, symbol Device:LED
- added R3, R4, R5, R6: R_US, Resistor_THT:R_Axial_DIN0207_L6.3mm_D2.5mm_P2.54mm_Vertical, symbol Device:R_US
- added U7: (no value), Library:ExBus_Edge, symbol New_Library_0:ExBus_Edge
- added U8: TS12A4515P, Package_DIP:DIP-8_W7.62mm, symbol Analog_Switch:ADG417BN
- R1, R2: footprint Resistor_THT:R_Axial_DIN0204_L3.6mm_D1.6mm_P7.62mm_Horizontal -> Resistor_THT:R_Axial_DIN0207_L6.3mm_D2.5mm_P2.54mm_Vertical
Connections:
- net CA2: now also U7.10 (CA2)
- net CB2: now also U7.12 (CB2)
- net GND: now also R6.1, U7.2 (GND)
- net PA6: now also R5.2, U8.1; no longer InRegHigh1.11 (SRCLK), InRegLow1.11 (SRCLK), PacketClockHigh1.5 (Q2), U6.11
- net PB0: now also U7.13 (PB0)
- net PB1: now also U7.14 (PB1)
- net PB2: now also U7.15 (PB2)
- net PB3: now also U7.16 (PB3)
- net PB4: now also U7.17 (PB4)
- net PB5: now also U7.18 (PB5)
- net PB6: now also U7.19 (PB6)
- net PB7: now also U7.20 (PB7)
- net VCC: now also R3.1, R4.1, U7.1 (VCC)
- net at U11.2: now also U7.5 (PA3)
- net at U11.5: now also U7.6 (PA4)
- net at U11.10: now also U7.7 (PA5)
- net at CONNPS2.1, InRegHigh1.14 (SER), U5.6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: now also R4.2
- net at U6.4: now also U8.6
- net at CONNPS2.5, U5.3: now also InRegHigh1.11 (SRCLK), InRegLow1.11 (SRCLK), U6.11, R3.2
- new net: D1.2 (A), PacketClockHigh1.5 (Q2), R5.1
- new net: D1.1 (K), R6.2
- new net: U7.8 (PA6), U8.8
Other:
- note removed: "Stack connector"
