File: Hardware/KiCad/avboard_tht2/Composite_Video_Generator.kicad_sch (KiCad schematic)
At the start: 58 parts, among them IC1 AS7C256C-15PCN, IC36 74HC4040, IC37 74HC30, IC39 74HC00, IC40 74HC4040, IC41 74HC00, IC43 74HC00, IC44 74HC86, IC45 74HC00, IC46 74HC257, IC47 74HC257, IC48 74HC564, IC53 74HC04, IC9 AS7C256C-15PCN, U2 THS7374, U3 74VHC373, U4 74VHC373, U5 74VHC373, U8 74HC244, U9 74HC244

Commit message: fix errors, reroute some things
Connections:
- net CHROMACARRIER: now also R10.2, R17.1, R18.1, R9.1; no longer R10.1, R12.1, R17.2, R18.2
- net GND: now also R16.2, R4.2; no longer R16.1, R4.1
- net at R11.2, R12.2, R13.1: now also R9.2; no longer R9.1
- net at R1.2, R5.1, R6.1: now also R4.1; no longer R4.2
- net at CHROMADAC0.3 (O): now also R10.1; no longer R10.2
- net at C3.-: now also R19.1; no longer R19.2
- net at C58.1, VIDJACK0.2: now also R19.2; no longer R19.1
- net at CHROMADAC0.6 (O): now also R12.1; no longer R9.2
- net at C2.2, R14.2, R15.2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: now also R16.1; no longer R16.2
- new net: C2.1, R17.2, R18.2
Other:
- moved on the sheet: R10, R12, R16, R17, R18, R19, R4, R9
Changed lines of the file:
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@@
 	)
 	(junction
-		(at 721.36 63.5)
-		(diameter 0)
-		(color 0 0 0 0)
-	)
-	(junction
 		(at 619.76 104.14)
 		(diameter 0)
@@
 	)
 	(junction
+		(at 617.22 104.14)
+		(diameter 0)
+		(color 0 0 0 0)
+	)
+	(junction
 		(at 71.12 294.64)
 		(diameter 0)
@@
 	)
 	(junction
+		(at 721.36 63.5)
+		(diameter 0)
+		(color 0 0 0 0)
+	)
+	(junction
 		(at 685.8 33.02)
 		(diameter 0)
@@
 	)
 	(junction
-		(at 617.22 104.14)
-		(diameter 0)
-		(color 0 0 0 0)
-	)
-	(junction
 		(at 552.45 337.82)
 		(diameter 0)
@@
 	(wire
 		(pts
-			(xy 721.36 63.5) (xy 721.36 66.04)
+			(xy 721.36 60.96) (xy 721.36 63.5)
 		)
 		(stroke
@@
 	(wire
 		(pts
+			(xy 721.36 63.5) (xy 721.36 66.04)
+		)
+		(stroke
+			(width 0.1524)
+			(type solid)
+		)
+	)
+	(wire
+		(pts
 			(xy 640.08 309.88) (xy 652.78 309.88)
 		)
@@
 	(wire
 		(pts
-			(xy 721.36 63.5) (xy 721.36 60.96)
-		)
-		(stroke
-			(width 0.1524)
-			(type solid)
-		)
-	)
-	(wire
-		(pts
 			(xy 290.83 152.4) (xy 331.47 152.4)
 		)
@@
 	(symbol
 		(lib_id "signals-eagle-import:R-US_0207/2V")
-		(at 723.9 71.12 90)
+		(at 716.28 63.5 0)
 		(unit 1)
 		(body_style 1)
@@
 		(dnp no)
 		(property "Reference" "R12"
-			(at 725.17 69.6214 90)
+			(at 716.28 59.944 0)
 			(show_name no)
 			(do_not_autoplace no)
@@
 		)
 		(property "Value" "1k"
-			(at 727.202 74.93 0)
+			(at 712.47 66.802 0)
 			(hide yes)
 			(show_name no)
@@
 		)
 		(property "Footprint" "Resistor_THT:R_Axial_DIN0207_L6.3mm_D2.5mm_P2.54mm_Vertical"
-			(at 723.9 71.12 0)
+			(at 716.28 63.5 0)
 			(hide yes)
 			(show_name no)
@@
 		)
 		(property "Datasheet" ""
-			(at 723.9 71.12 0)
+			(at 716.28 63.5 0)
 			(hide yes)
 			(show_name no)
@@
 		)
 		(property "Description" ""
-			(at 723.9 71.12 0)
+			(at 716.28 63.5 0)
 			(show_name no)
 			(do_not_autoplace no)
@@
 		)
 		(property "MPN" "tbd"
-			(at 723.9 71.12 0)
+			(at 716.28 63.5 0)
 			(hide yes)
 			(show_name no)
@@
 		)
 		(property "Manufacturer_Part_Number" ""
-			(at 723.9 71.12 90)
+			(at 716.28 63.5 90)
 			(hide yes)
 			(show_name no)
@@
 		)
 		(property "THT" "yes"
-			(at 723.9 71.12 90)
+			(at 716.28 63.5 90)
 			(hide yes)
 			(show_name no)
@@
 	(symbol
 		(lib_id "signals-eagle-import:R-US_0207/2V")
-		(at 716.28 78.74 180)
+		(at 716.28 78.74 0)
 		(unit 1)
 		(body_style 1)
@@
 		(dnp no)
 		(property "Reference" "R10"
-			(at 720.09 80.2386 0)
+			(at 712.47 77.2414 0)
 			(show_name no)
 			(do_not_autoplace no)
@@
 		)
 		(property "Value" "1k"
-			(at 720.09 75.438 0)
+			(at 712.47 82.042 0)
 			(hide yes)
 			(show_name no)
@@
 	(symbol
 		(lib_id "signals-eagle-import:R-US_0204/7")
-		(at 723.9 88.9 90)
+		(at 718.82 88.9 270)
 		(unit 1)
 		(body_style 1)
@@
 		(dnp no)
 		(property "Reference" "R18"
-			(at 730.0214 92.71 0)
+			(at 712.6986 85.09 0)
 			(show_name no)
 			(do_not_autoplace no)
@@
 		)
 		(property "Value" "3.3k"
-			(at 727.202 92.71 0)
+			(at 715.518 85.09 0)
 			(show_name no)
 			(do_not_autoplace no)
@@
 		)
 		(property "Footprint" "Resistor_THT:R_Axial_DIN0207_L6.3mm_D2.5mm_P2.54mm_Vertical"
-			(at 723.9 88.9 0)
+			(at 718.82 88.9 0)
 			(hide yes)
 			(show_name no)
@@
 		)
 		(property "Datasheet" ""
-			(at 723.9 88.9 0)
+			(at 718.82 88.9 0)
 			(hide yes)
 			(show_name no)
@@
 		)
 		(property "Description" ""
-			(at 723.9 88.9 0)
+			(at 718.82 88.9 0)
 			(show_name no)
 			(do_not_autoplace no)
@@
 		)
 		(property "MPN" "tbd"
-			(at 723.9 88.9 0)
+			(at 718.82 88.9 0)
 			(hide yes)
 			(show_name no)
@@
 		)
 		(property "Manufacturer_Part_Number" ""
-			(at 723.9 88.9 0)
+			(at 718.82 88.9 0)
 			(hide yes)
 			(show_name no)
@@
 		)
 		(property "THT" "yes"
-			(at 723.9 88.9 0)
+			(at 718.82 88.9 0)
 			(hide yes)
 			(show_name no)
@@
 	(symbol
 		(lib_id "signals-eagle-import:R-US_0204/7")
-		(at 731.52 114.3 90)
+		(at 731.52 114.3 270)
 		(unit 1)
 		(body_style 1)
@@
 		(dnp no)
 		(property "Reference" "R16"
-			(at 730.0214 118.11 0)
+			(at 728.218 110.49 0)
 			(show_name no)
 			(do_not_autoplace no)
@@
 		)
 		(property "Value" "150"
-			(at 734.822 118.11 0)
+			(at 733.0186 110.49 0)
 			(show_name no)
 			(do_not_autoplace no)
@@
 	(symbol
 		(lib_id "signals-eagle-import:R-US_0207/2V")
-		(at 716.28 63.5 180)
+		(at 723.9 71.12 90)
 		(unit 1)
 		(body_style 1)
@@
 		(dnp no)
 		(property "Reference" "R9"
-			(at 720.09 64.9986 0)
+			(at 722.4014 74.93 0)
 			(show_name no)
 			(do_not_autoplace no)
@@
 		)
 		(property "Value" "1k"
-			(at 720.09 60.198 0)
+			(at 727.202 74.93 0)
 			(hide yes)
 			(show_name no)
@@
 		)
 		(property "Footprint" "Resistor_THT:R_Axial_DIN0207_L6.3mm_D2.5mm_P2.54mm_Vertical"
-			(at 716.28 63.5 0)
+			(at 723.9 71.12 0)
 			(hide yes)
 			(show_name no)
@@
 		)
 		(property "Datasheet" ""
-			(at 716.28 63.5 0)
+			(at 723.9 71.12 0)
 			(hide yes)
 			(show_name no)
@@
 		)
 		(property "Description" ""
-			(at 716.28 63.5 0)
+			(at 723.9 71.12 0)
 			(show_name no)
 			(do_not_autoplace no)
@@
 		)
 		(property "MPN" "tbd"
-			(at 716.28 63.5 0)
+			(at 723.9 71.12 0)
 			(hide yes)
 			(show_name no)
@@
 		)
 		(property "Manufacturer_Part_Number" ""
-			(at 716.28 63.5 0)
+			(at 723.9 71.12 0)
 			(hide yes)
 			(show_name no)
@@
 		)
 		(property "THT" "yes"
-			(at 716.28 63.5 0)
+			(at 723.9 71.12 0)
 			(hide yes)
 			(show_name no)
@@
 	(symbol
 		(lib_id "signals-eagle-import:R-US_0204/7")
-		(at 718.82 88.9 90)
+		(at 723.9 88.9 270)
 		(unit 1)
 		(body_style 1)
@@
 		(dnp no)
 		(property "Reference" "R17"
-			(at 717.3214 92.71 0)
+			(at 725.3986 85.09 0)
 			(show_name no)
 			(do_not_autoplace no)
@@
 		)
 		(property "Value" "3.3k"
-			(at 714.502 92.71 0)
+			(at 728.218 85.09 0)
 			(show_name no)
 			(do_not_autoplace no)
@@
 		)
 		(property "Footprint" "Resistor_THT:R_Axial_DIN0207_L6.3mm_D2.5mm_P2.54mm_Vertical"
-			(at 718.82 88.9 0)
+			(at 723.9 88.9 0)
 			(hide yes)
 			(show_name no)
@@
 		)
 		(property "Datasheet" ""
-			(at 718.82 88.9 0)
+			(at 723.9 88.9 0)
 			(hide yes)
 			(show_name no)
@@
 		)
 		(property "Description" ""
-			(at 718.82 88.9 0)
+			(at 723.9 88.9 0)
 			(show_name no)
 			(do_not_autoplace no)
@@
 		)
 		(property "MPN" "tbd"
-			(at 718.82 88.9 0)
+			(at 723.9 88.9 0)
 			(hide yes)
 			(show_name no)
@@
 		)
 		(property "Manufacturer_Part_Number" ""
-			(at 718.82 88.9 0)
+			(at 723.9 88.9 0)
 			(hide yes)
 			(show_name no)
@@
 		)
 		(property "THT" "yes"
-			(at 718.82 88.9 0)
+			(at 723.9 88.9 0)
 			(hide yes)
 			(show_name no)
@@
 	(symbol
 		(lib_id "signals-eagle-import:R-US_0204/7")
-		(at 836.93 104.14 180)
+		(at 836.93 104.14 0)
 		(unit 1)
 		(body_style 1)
@@
 		(dnp no)
 		(property "Reference" "R19"
-			(at 835.66 100.5586 0)
+			(at 832.866 102.108 0)
 			(show_name no)
 			(do_not_autoplace no)
@@
 		)
 		(property "Value" "75"
-			(at 840.74 100.838 0)
+			(at 838.454 102.616 0)
 			(show_name no)
 			(do_not_autoplace no)
@@
 	(symbol
 		(lib_id "signals-eagle-import:R-US_0207/2V")
-		(at 612.14 104.14 0)
+		(at 612.14 104.14 180)
 		(unit 1)
 		(body_style 1)
@@
 		(dnp no)
 		(property "Reference" "R4"
-			(at 608.33 102.6414 0)
+			(at 610.87 100.838 0)
 			(show_name no)
 			(do_not_autoplace no)
@@
 		)
 		(property "Value" "1k"
-			(at 608.33 107.442 0)
+			(at 615.95 100.838 0)
 			(hide yes)
 			(show_name no)
