File: Hardware/KiCad/avboard_tht2/signals_4.kicad_sch (KiCad schematic)
At the start: 22 parts, among them IC2_AUD0 74HC32, IC4_AUD0 74HC00, IC6_AUD0 74HC74, IC7_AUD0 LM358N, U1 W65C02S

Commit message: fix SysD7 bug and a few tracing improvements
Connections:
- net AR/~{W}B: now also IC2_AUD0.13 (I1); no longer IC2_AUD0.10 (I1)
- net SysD6: no longer J6.33
- net SysD7: now also J6.33
- net at IC4_AUD0.3 (O): now also IC2_AUD0.12 (I0); no longer IC2_AUD0.9 (I0)
- net at IC4_AUD0.4 (I0), IC4_AUD0.5 (I1): now also IC2_AUD0.11 (O); no longer IC2_AUD0.8 (O)
Changed lines of the file:
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@@
 		)
 	)
-	(label "SysD6"
+	(label "SysD7"
 		(at 118.11 29.21 270)
 		(effects
@@
 		(lib_id "signals-eagle-import:7432N")
 		(at 322.58 121.92 90)
-		(unit 3)
+		(unit 4)
 		(body_style 1)
 		(exclude_from_sim no)
@@
 				(path "/ecfc5df0-38b0-48e8-a960-6f082396f7df/37ec6fca-c60e-4524-9a8e-c3db557ac388"
 					(reference "IC2_AUD0")
-					(unit 3)
+					(unit 4)
 				)
 			)

Commit message: fix errors, reroute some things
Connections:
- net AUDIO_RDY: now also R21.2; no longer R21.1
- net at U1.2 (RDY): now also R21.1; no longer R21.2
Other:
- moved on the sheet: R21
Changed lines of the file:
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@@
 	(symbol
 		(lib_id "signals-eagle-import:R-US_0207/10")
-		(at 231.14 198.12 0)
+		(at 231.14 198.12 180)
 		(unit 1)
 		(body_style 1)
@@
 		(dnp no)
 		(property "Reference" "R21"
-			(at 227.33 196.6214 0)
+			(at 234.95 194.818 0)
 			(show_name no)
 			(do_not_autoplace no)
@@
 		)
 		(property "Value" "3.3k"
-			(at 227.33 201.422 0)
+			(at 234.95 199.6186 0)
 			(show_name no)
 			(do_not_autoplace no)
